File: hardware/mega/atari2600-cart-reader-mega.kicad_sch (KiCad schematic)
At the start: 4 parts, among them J1 Atari 2600 Cartridge-Slot

Commit message: Set cartridge slot row spacing to measured 5.5 mm
Stefan measured 6 mm across the outer pin edges with 0.5 mm pins.
Both shields re-routed; DRC 0 errors, 0 unconnected.

Co-Authored-By: Claude Opus 5.5 (1M context) <noreply@anthropic.com>
Claude-Session: https://claude.ai/code/session_015VQCpzuZ22TPQEmx9cLrbH
Parts:
- J1: footprint atari:Atari2600_Cart_Slot_2x12_P2.54mm_Row5.08mm -> atari:Atari2600_Cart_Slot_2x12_P2.54mm_Row5.50mm
Changed lines of the file:
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@@
     (instances
       (project "atari2600-cart-reader-mega"
-        (path "/4d6e53de-9d56-47f0-a5e5-ce794cd93521"
+        (path "/ce326073-864b-4a1d-b07c-58e5fa503181"
           (reference "A1")
           (unit 1)))))
@@
     (instances
       (project "atari2600-cart-reader-mega"
-        (path "/4d6e53de-9d56-47f0-a5e5-ce794cd93521"
+        (path "/ce326073-864b-4a1d-b07c-58e5fa503181"
           (reference "#PWR01")
           (unit 1)))))
@@
     (instances
       (project "atari2600-cart-reader-mega"
-        (path "/4d6e53de-9d56-47f0-a5e5-ce794cd93521"
+        (path "/ce326073-864b-4a1d-b07c-58e5fa503181"
           (reference "#PWR02")
           (unit 1)))))
@@
     (instances
       (project "atari2600-cart-reader-mega"
-        (path "/4d6e53de-9d56-47f0-a5e5-ce794cd93521"
+        (path "/ce326073-864b-4a1d-b07c-58e5fa503181"
           (reference "#PWR03")
           (unit 1)))))
@@
     (instances
       (project "atari2600-cart-reader-mega"
-        (path "/4d6e53de-9d56-47f0-a5e5-ce794cd93521"
+        (path "/ce326073-864b-4a1d-b07c-58e5fa503181"
           (reference "#PWR04")
           (unit 1)))))
@@
     (instances
       (project "atari2600-cart-reader-mega"
-        (path "/4d6e53de-9d56-47f0-a5e5-ce794cd93521"
+        (path "/ce326073-864b-4a1d-b07c-58e5fa503181"
           (reference "#PWR05")
           (unit 1)))))
@@
     (instances
       (project "atari2600-cart-reader-mega"
-        (path "/4d6e53de-9d56-47f0-a5e5-ce794cd93521"
+        (path "/ce326073-864b-4a1d-b07c-58e5fa503181"
           (reference "#PWR06")
           (unit 1)))))
@@
     (instances
       (project "atari2600-cart-reader-mega"
-        (path "/4d6e53de-9d56-47f0-a5e5-ce794cd93521"
+        (path "/ce326073-864b-4a1d-b07c-58e5fa503181"
           (reference "#PWR07")
           (unit 1)))))
@@
     (instances
       (project "atari2600-cart-reader-mega"
-        (path "/4d6e53de-9d56-47f0-a5e5-ce794cd93521"
+        (path "/ce326073-864b-4a1d-b07c-58e5fa503181"
           (reference "#PWR08")
           (unit 1)))))
@@
         (font
           (size 1.27 1.27))))
-    (property "Footprint" "atari:Atari2600_Cart_Slot_2x12_P2.54mm_Row5.08mm"
+    (property "Footprint" "atari:Atari2600_Cart_Slot_2x12_P2.54mm_Row5.50mm"
       (at 215 100 0)
       (effects
@@
     (instances
       (project "atari2600-cart-reader-mega"
-        (path "/4d6e53de-9d56-47f0-a5e5-ce794cd93521"
+        (path "/ce326073-864b-4a1d-b07c-58e5fa503181"
           (reference "J1")
           (unit 1)))))
@@
     (instances
       (project "atari2600-cart-reader-mega"
-        (path "/4d6e53de-9d56-47f0-a5e5-ce794cd93521"
+        (path "/ce326073-864b-4a1d-b07c-58e5fa503181"
           (reference "#PWR09")
           (unit 1)))))
@@
     (instances
       (project "atari2600-cart-reader-mega"
-        (path "/4d6e53de-9d56-47f0-a5e5-ce794cd93521"
+        (path "/ce326073-864b-4a1d-b07c-58e5fa503181"
           (reference "#PWR10")
           (unit 1)))))
@@
     (instances
       (project "atari2600-cart-reader-mega"
-        (path "/4d6e53de-9d56-47f0-a5e5-ce794cd93521"
+        (path "/ce326073-864b-4a1d-b07c-58e5fa503181"
           (reference "#PWR11")
           (unit 1)))))
@@
     (instances
       (project "atari2600-cart-reader-mega"
-        (path "/4d6e53de-9d56-47f0-a5e5-ce794cd93521"
+        (path "/ce326073-864b-4a1d-b07c-58e5fa503181"
           (reference "C2")
           (unit 1)))))
@@
     (instances
       (project "atari2600-cart-reader-mega"
-        (path "/4d6e53de-9d56-47f0-a5e5-ce794cd93521"
+        (path "/ce326073-864b-4a1d-b07c-58e5fa503181"
           (reference "#PWR12")
           (unit 1)))))
@@
     (instances
       (project "atari2600-cart-reader-mega"
-        (path "/4d6e53de-9d56-47f0-a5e5-ce794cd93521"
+        (path "/ce326073-864b-4a1d-b07c-58e5fa503181"
           (reference "#PWR13")
           (unit 1)))))
@@
     (instances
       (project "atari2600-cart-reader-mega"
-        (path "/4d6e53de-9d56-47f0-a5e5-ce794cd93521"
+        (path "/ce326073-864b-4a1d-b07c-58e5fa503181"
           (reference "C3")
           (unit 1)))))
@@
     (instances
       (project "atari2600-cart-reader-mega"
-        (path "/4d6e53de-9d56-47f0-a5e5-ce794cd93521"
+        (path "/ce326073-864b-4a1d-b07c-58e5fa503181"
           (reference "#PWR14")
           (unit 1)))))
@@
     (instances
       (project "atari2600-cart-reader-mega"
-        (path "/4d6e53de-9d56-47f0-a5e5-ce794cd93521"
+        (path "/ce326073-864b-4a1d-b07c-58e5fa503181"
           (reference "#PWR15")
           (unit 1)))))
@@
     (instances
       (project "atari2600-cart-reader-mega"
-        (path "/4d6e53de-9d56-47f0-a5e5-ce794cd93521"
+        (path "/ce326073-864b-4a1d-b07c-58e5fa503181"
           (reference "#FLG01")
           (unit 1)))))
@@
     (instances
       (project "atari2600-cart-reader-mega"
-        (path "/4d6e53de-9d56-47f0-a5e5-ce794cd93521"
+        (path "/ce326073-864b-4a1d-b07c-58e5fa503181"
           (reference "#PWR17")
           (unit 1)))))
@@
     (instances
       (project "atari2600-cart-reader-mega"
-        (path "/4d6e53de-9d56-47f0-a5e5-ce794cd93521"
+        (path "/ce326073-864b-4a1d-b07c-58e5fa503181"
           (reference "#FLG02")
           (unit 1)))))
@@
     (instances
       (project "atari2600-cart-reader-mega"
-        (path "/4d6e53de-9d56-47f0-a5e5-ce794cd93521"
+        (path "/ce326073-864b-4a1d-b07c-58e5fa503181"
           (reference "#PWR19")
           (unit 1)))))

Commit message: Switched cartridge supply, Nano board, guide mounting holes
- BC327 high-side switch with 200 mA polyfuse and rail sense on all boards
- Firmware powers the cartridge only after an orientation check
  (experimental thresholds, S command for calibration)
- New carrier board for a plugged-in Arduino Nano (same circuit and
  firmware as the Uno)
- Slot footprint with M2.5 flange holes and the guide base plate outline;
  build checks that the plate area stays free
- ICSP header removed from the shields, Uno hole next to it removed,
  Mega slot moved to the board centre
- Fix: struct Scheme declared before Arduino's generated prototypes
  (the sketch did not compile before)
- Switch schematic and prototype photos

Co-Authored-By: Claude Opus 5.5 (1M context) <noreply@anthropic.com>
Claude-Session: https://claude.ai/code/session_015VQCpzuZ22TPQEmx9cLrbH
Parts:
- added F1: MF-R020 (200 mA), atari:Fuse_PTC_Radial_P5.08mm, symbol Device:Polyfuse
- added Q1: BC327, Package_TO_SOT_THT:TO-92_Inline, symbol Transistor_BJT:BC327
- added R3: 1k, Resistor_THT:R_Axial_DIN0207_L6.3mm_D2.5mm_P7.62mm_Horizontal, symbol Device:R
- added R4, R5: 10k, Resistor_THT:R_Axial_DIN0207_L6.3mm_D2.5mm_P7.62mm_Horizontal, symbol Device:R
- added R6: 100k, Resistor_THT:R_Axial_DIN0207_L6.3mm_D2.5mm_P7.62mm_Horizontal, symbol Device:R
- J1: footprint atari:Atari2600_Cart_Slot_2x12_P2.54mm_Row5.50mm -> atari:Atari2600_Cart_Slot_2x12_P2.54mm_Row5.50mm_Guide
Connections:
- net +5V: now also F1.1; no longer C2.1, J1.23 (Pin_23)
- net GND: now also R6.2
- net CART_SENSE: now reaches A1.A0
- net CART_SENSE: now also R5.2
- net CART_PWR: now reaches A1.D8
- net CART_PWR: now also R3.1
- new net +5V_F: F1.2, Q1.3 (E), R4.1
- new net CART_5V: C2.1, J1.23 (Pin_23), Q1.1 (C), R5.1, R6.1
- new net Q_BASE: Q1.2 (B), R3.2, R4.2
- no-connect marks 62 -> 60

Commit message: Reset and read buttons on all boards (v1.2)
SW1 resets the Arduino, SW2 on A1 repeats the last dump; dump.py listen saves button dumps.

Co-Authored-By: Claude Opus 5.5 <noreply@anthropic.com>
Claude-Session: https://claude.ai/code/session_015VQCpzuZ22TPQEmx9cLrbH
Parts:
- added SW1: Reset, Button_Switch_THT:SW_PUSH_6mm, symbol Switch:SW_Push
- added SW2: Read, Button_Switch_THT:SW_PUSH_6mm, symbol Switch:SW_Push
Connections:
- net GND: now also SW1.2, SW2.2
- net READ: now reaches A1.A1
- net READ: now also SW2.1
- net RESET: now reaches A1.RST1 (RESET)
- net RESET: now also SW1.1
- no-connect marks 60 -> 58
