File: hardware/nano/atari2600-cart-reader-nano.kicad_sch (KiCad schematic)
At the start: 16 parts, among them J1 Atari 2600 Cartridge-Slot, Q1 BC327, U1 MCP23017-E/SP

Commit message: Reset and read buttons on all boards (v1.2)
SW1 resets the Arduino, SW2 on A1 repeats the last dump; dump.py listen saves button dumps.

Co-Authored-By: Claude Opus 5.5 <noreply@anthropic.com>
Claude-Session: https://claude.ai/code/session_015VQCpzuZ22TPQEmx9cLrbH
Parts:
- added SW1: Reset, Button_Switch_THT:SW_PUSH_6mm, symbol Switch:SW_Push
- added SW2: Read, Button_Switch_THT:SW_PUSH_6mm, symbol Switch:SW_Push
Connections:
- net GND: now also SW1.2, SW2.2
- net READ: now reaches A1.20 (A1)
- net READ: now also SW2.1
- net RESET: now reaches A1.3 (~{RESET})
- net RESET: now also SW1.1
- no-connect marks 22 -> 20

Commit message: Nano board: read button only, the Nano's own reset button stays reachable
Co-Authored-By: Claude Opus 5.5 <noreply@anthropic.com>
Claude-Session: https://claude.ai/code/session_015VQCpzuZ22TPQEmx9cLrbH
Parts:
- removed SW1: Reset, Button_Switch_THT:SW_PUSH_6mm, symbol Switch:SW_Push
Connections:
- net RESET: no longer names the net of A1.3 (~{RESET})
- no-connect marks 20 -> 21

Commit message: Uno/Nano: address bus via two 74HC595 on SPI, MCP23017 boards kept as variants
hal.h selects the MCP23017 with #define ADDR_MCP23017.

Co-Authored-By: Claude Opus 5.5 <noreply@anthropic.com>
Claude-Session: https://claude.ai/code/session_015VQCpzuZ22TPQEmx9cLrbH
Parts:
- removed R1, R2: 4k7, Resistor_THT:R_Axial_DIN0207_L6.3mm_D2.5mm_P7.62mm_Horizontal, symbol Device:R
- removed U1: MCP23017-E/SP, Package_DIP:DIP-28_W7.62mm_Socket, symbol Interface_Expansion:MCP23017_SP
- added C4: 100n, Capacitor_THT:C_Disc_D5.0mm_W2.5mm_P5.00mm, symbol Device:C
- added U1, U2: 74HC595, Package_DIP:DIP-16_W7.62mm_Socket, symbol 74xx:74HC595
Connections:
- net +5V: now also C4.1, U1.10 (~{SRCLR}), U1.16 (VCC), U2.10 (~{SRCLR}), U2.16 (VCC)
- net A0: now also U1.15 (QA)
- net A1: now also U1.1 (QB)
- net A10: now also U2.2 (QC)
- net A11: now also U2.3 (QD)
- net A12: now also U2.4 (QE)
- net A2: now also U1.2 (QC)
- net A3: now also U1.3 (QD)
- net A4: now also U1.4 (QE)
- net A5: now also U1.5 (QF)
- net A6: now also U1.6 (QG)
- net A7: now also U1.7 (QH)
- net A8: now also U2.15 (QA)
- net A9: now also U2.1 (QB)
- net GND: now also C4.2, U1.13 (~{OE}), U1.8 (GND), U2.13 (~{OE}), U2.8 (GND)
- net MOSI: now reaches A1.14 (D11)
- net MOSI: now also U1.14 (SER)
- net SCK: now reaches A1.16 (D13)
- net SCK: now also U1.11 (SRCLK), U2.11 (SRCLK)
- net LATCH: now reaches A1.21 (A2)
- net LATCH: now also U1.12 (RCLK), U2.12 (RCLK)
- net SCL: no longer names the net of A1.24 (A5)
- net SDA: no longer names the net of A1.23 (A4)
- new net SR_CHAIN: U1.9 (QH'), U2.14 (SER)
- no-connect marks 21 -> 17
Other:
- note added: "Traegerplatine fuer Arduino Nano (ATmega328P, gesteckt). Gleiche Belegung und Firmware wie die Uno-Variante: Adressbus A0-A12 ueber 2x 74HC595 (SPI: D11, D13, Latch A2), Datenbus D0-D7 an Nano D2-D9, Versorgung Cartridge D10, Messung A0. Firmware: github.com/sfambach/arduino-atari2600-cart-reader - fambach.net"
- note removed: "Traegerplatine fuer Arduino Nano (ATmega328P, gesteckt). Gleiche Belegung und Firmware wie die Uno-Variante: Adressbus A0-A12 ueber MCP23017 (I2C 0x20), Datenbus D0-D7 an Nano D2-D9, Versorgung Cartridge D10, Messung A0. Firmware: github.com/sfambach/arduino-atari2600-cart-reader - fambach.net"
