File: hardware/uno/atari2600-cart-reader-uno.kicad_sch (KiCad schematic)
At the start: 8 parts, among them J1 Atari 2600 Cartridge-Slot, U1 MCP23017-E/SP

Commit message: Set cartridge slot row spacing to measured 5.5 mm
Stefan measured 6 mm across the outer pin edges with 0.5 mm pins.
Both shields re-routed; DRC 0 errors, 0 unconnected.

Co-Authored-By: Claude Opus 5.5 (1M context) <noreply@anthropic.com>
Claude-Session: https://claude.ai/code/session_015VQCpzuZ22TPQEmx9cLrbH
Parts:
- J1: footprint atari:Atari2600_Cart_Slot_2x12_P2.54mm_Row5.08mm -> atari:Atari2600_Cart_Slot_2x12_P2.54mm_Row5.50mm
Changed lines of the file:
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@@
     (instances
       (project "atari2600-cart-reader-uno"
-        (path "/7ce413c0-2e94-4054-afd6-e7ae1bf55d48"
+        (path "/49daac6a-64be-44f1-b946-f1c4c9283681"
           (reference "A1")
           (unit 1)))))
@@
     (instances
       (project "atari2600-cart-reader-uno"
-        (path "/7ce413c0-2e94-4054-afd6-e7ae1bf55d48"
+        (path "/49daac6a-64be-44f1-b946-f1c4c9283681"
           (reference "#PWR01")
           (unit 1)))))
@@
     (instances
       (project "atari2600-cart-reader-uno"
-        (path "/7ce413c0-2e94-4054-afd6-e7ae1bf55d48"
+        (path "/49daac6a-64be-44f1-b946-f1c4c9283681"
           (reference "#PWR02")
           (unit 1)))))
@@
     (instances
       (project "atari2600-cart-reader-uno"
-        (path "/7ce413c0-2e94-4054-afd6-e7ae1bf55d48"
+        (path "/49daac6a-64be-44f1-b946-f1c4c9283681"
           (reference "#PWR03")
           (unit 1)))))
@@
     (instances
       (project "atari2600-cart-reader-uno"
-        (path "/7ce413c0-2e94-4054-afd6-e7ae1bf55d48"
+        (path "/49daac6a-64be-44f1-b946-f1c4c9283681"
           (reference "#PWR04")
           (unit 1)))))
@@
         (font
           (size 1.27 1.27))))
-    (property "Footprint" "atari:Atari2600_Cart_Slot_2x12_P2.54mm_Row5.08mm"
+    (property "Footprint" "atari:Atari2600_Cart_Slot_2x12_P2.54mm_Row5.50mm"
       (at 215 100 0)
       (effects
@@
     (instances
       (project "atari2600-cart-reader-uno"
-        (path "/7ce413c0-2e94-4054-afd6-e7ae1bf55d48"
+        (path "/49daac6a-64be-44f1-b946-f1c4c9283681"
           (reference "J1")
           (unit 1)))))
@@
     (instances
       (project "atari2600-cart-reader-uno"
-        (path "/7ce413c0-2e94-4054-afd6-e7ae1bf55d48"
+        (path "/49daac6a-64be-44f1-b946-f1c4c9283681"
           (reference "#PWR05")
           (unit 1)))))
@@
     (instances
       (project "atari2600-cart-reader-uno"
-        (path "/7ce413c0-2e94-4054-afd6-e7ae1bf55d48"
+        (path "/49daac6a-64be-44f1-b946-f1c4c9283681"
           (reference "#PWR06")
           (unit 1)))))
@@
     (instances
       (project "atari2600-cart-reader-uno"
-        (path "/7ce413c0-2e94-4054-afd6-e7ae1bf55d48"
+        (path "/49daac6a-64be-44f1-b946-f1c4c9283681"
           (reference "#PWR07")
           (unit 1)))))
@@
     (instances
       (project "atari2600-cart-reader-uno"
-        (path "/7ce413c0-2e94-4054-afd6-e7ae1bf55d48"
+        (path "/49daac6a-64be-44f1-b946-f1c4c9283681"
           (reference "U1")
           (unit 1)))))
@@
     (instances
       (project "atari2600-cart-reader-uno"
-        (path "/7ce413c0-2e94-4054-afd6-e7ae1bf55d48"
+        (path "/49daac6a-64be-44f1-b946-f1c4c9283681"
           (reference "#PWR08")
           (unit 1)))))
@@
     (instances
       (project "atari2600-cart-reader-uno"
-        (path "/7ce413c0-2e94-4054-afd6-e7ae1bf55d48"
+        (path "/49daac6a-64be-44f1-b946-f1c4c9283681"
           (reference "#PWR09")
           (unit 1)))))
@@
     (instances
       (project "atari2600-cart-reader-uno"
-        (path "/7ce413c0-2e94-4054-afd6-e7ae1bf55d48"
+        (path "/49daac6a-64be-44f1-b946-f1c4c9283681"
           (reference "#PWR10")
           (unit 1)))))
@@
     (instances
       (project "atari2600-cart-reader-uno"
-        (path "/7ce413c0-2e94-4054-afd6-e7ae1bf55d48"
+        (path "/49daac6a-64be-44f1-b946-f1c4c9283681"
           (reference "#PWR11")
           (unit 1)))))
@@
     (instances
       (project "atari2600-cart-reader-uno"
-        (path "/7ce413c0-2e94-4054-afd6-e7ae1bf55d48"
+        (path "/49daac6a-64be-44f1-b946-f1c4c9283681"
           (reference "#PWR12")
           (unit 1)))))
@@
     (instances
       (project "atari2600-cart-reader-uno"
-        (path "/7ce413c0-2e94-4054-afd6-e7ae1bf55d48"
+        (path "/49daac6a-64be-44f1-b946-f1c4c9283681"
           (reference "#PWR13")
           (unit 1)))))
@@
     (instances
       (project "atari2600-cart-reader-uno"
-        (path "/7ce413c0-2e94-4054-afd6-e7ae1bf55d48"
+        (path "/49daac6a-64be-44f1-b946-f1c4c9283681"
           (reference "R1")
           (unit 1)))))
@@
     (instances
       (project "atari2600-cart-reader-uno"
-        (path "/7ce413c0-2e94-4054-afd6-e7ae1bf55d48"
+        (path "/49daac6a-64be-44f1-b946-f1c4c9283681"
           (reference "#PWR14")
           (unit 1)))))
@@
     (instances
       (project "atari2600-cart-reader-uno"
-        (path "/7ce413c0-2e94-4054-afd6-e7ae1bf55d48"
+        (path "/49daac6a-64be-44f1-b946-f1c4c9283681"
           (reference "R2")
           (unit 1)))))
@@
     (instances
       (project "atari2600-cart-reader-uno"
-        (path "/7ce413c0-2e94-4054-afd6-e7ae1bf55d48"
+        (path "/49daac6a-64be-44f1-b946-f1c4c9283681"
           (reference "#PWR15")
           (unit 1)))))
@@
     (instances
       (project "atari2600-cart-reader-uno"
-        (path "/7ce413c0-2e94-4054-afd6-e7ae1bf55d48"
+        (path "/49daac6a-64be-44f1-b946-f1c4c9283681"
           (reference "C1")
           (unit 1)))))
@@
     (instances
       (project "atari2600-cart-reader-uno"
-        (path "/7ce413c0-2e94-4054-afd6-e7ae1bf55d48"
+        (path "/49daac6a-64be-44f1-b946-f1c4c9283681"
           (reference "#PWR16")
           (unit 1)))))
@@
     (instances
       (project "atari2600-cart-reader-uno"
-        (path "/7ce413c0-2e94-4054-afd6-e7ae1bf55d48"
+        (path "/49daac6a-64be-44f1-b946-f1c4c9283681"
           (reference "#PWR17")
           (unit 1)))))
@@
     (instances
       (project "atari2600-cart-reader-uno"
-        (path "/7ce413c0-2e94-4054-afd6-e7ae1bf55d48"
+        (path "/49daac6a-64be-44f1-b946-f1c4c9283681"
           (reference "C2")
           (unit 1)))))
@@
     (instances
       (project "atari2600-cart-reader-uno"
-        (path "/7ce413c0-2e94-4054-afd6-e7ae1bf55d48"
+        (path "/49daac6a-64be-44f1-b946-f1c4c9283681"
           (reference "#PWR18")
           (unit 1)))))
@@
     (instances
       (project "atari2600-cart-reader-uno"
-        (path "/7ce413c0-2e94-4054-afd6-e7ae1bf55d48"
+        (path "/49daac6a-64be-44f1-b946-f1c4c9283681"
           (reference "#PWR19")
           (unit 1)))))
@@
     (instances
       (project "atari2600-cart-reader-uno"
-        (path "/7ce413c0-2e94-4054-afd6-e7ae1bf55d48"
+        (path "/49daac6a-64be-44f1-b946-f1c4c9283681"
           (reference "C3")
           (unit 1)))))
@@
     (instances
       (project "atari2600-cart-reader-uno"
-        (path "/7ce413c0-2e94-4054-afd6-e7ae1bf55d48"
+        (path "/49daac6a-64be-44f1-b946-f1c4c9283681"
           (reference "#PWR20")
           (unit 1)))))
@@
     (instances
       (project "atari2600-cart-reader-uno"
-        (path "/7ce413c0-2e94-4054-afd6-e7ae1bf55d48"
+        (path "/49daac6a-64be-44f1-b946-f1c4c9283681"
           (reference "#PWR21")
           (unit 1)))))
@@
     (instances
       (project "atari2600-cart-reader-uno"
-        (path "/7ce413c0-2e94-4054-afd6-e7ae1bf55d48"
+        (path "/49daac6a-64be-44f1-b946-f1c4c9283681"
           (reference "#FLG01")
           (unit 1)))))
@@
     (instances
       (project "atari2600-cart-reader-uno"
-        (path "/7ce413c0-2e94-4054-afd6-e7ae1bf55d48"
+        (path "/49daac6a-64be-44f1-b946-f1c4c9283681"
           (reference "#PWR23")
           (unit 1)))))
@@
     (instances
       (project "atari2600-cart-reader-uno"
-        (path "/7ce413c0-2e94-4054-afd6-e7ae1bf55d48"
+        (path "/49daac6a-64be-44f1-b946-f1c4c9283681"
           (reference "#FLG02")
           (unit 1)))))
@@
     (instances
       (project "atari2600-cart-reader-uno"
-        (path "/7ce413c0-2e94-4054-afd6-e7ae1bf55d48"
+        (path "/49daac6a-64be-44f1-b946-f1c4c9283681"
           (reference "#PWR25")
           (unit 1)))))

Commit message: Switched cartridge supply, Nano board, guide mounting holes
- BC327 high-side switch with 200 mA polyfuse and rail sense on all boards
- Firmware powers the cartridge only after an orientation check
  (experimental thresholds, S command for calibration)
- New carrier board for a plugged-in Arduino Nano (same circuit and
  firmware as the Uno)
- Slot footprint with M2.5 flange holes and the guide base plate outline;
  build checks that the plate area stays free
- ICSP header removed from the shields, Uno hole next to it removed,
  Mega slot moved to the board centre
- Fix: struct Scheme declared before Arduino's generated prototypes
  (the sketch did not compile before)
- Switch schematic and prototype photos

Co-Authored-By: Claude Opus 5.5 (1M context) <noreply@anthropic.com>
Claude-Session: https://claude.ai/code/session_015VQCpzuZ22TPQEmx9cLrbH
Parts:
- added F1: MF-R020 (200 mA), atari:Fuse_PTC_Radial_P5.08mm, symbol Device:Polyfuse
- added Q1: BC327, Package_TO_SOT_THT:TO-92_Inline, symbol Transistor_BJT:BC327
- added R3: 1k, Resistor_THT:R_Axial_DIN0207_L6.3mm_D2.5mm_P7.62mm_Horizontal, symbol Device:R
- added R4, R5: 10k, Resistor_THT:R_Axial_DIN0207_L6.3mm_D2.5mm_P7.62mm_Horizontal, symbol Device:R
- added R6: 100k, Resistor_THT:R_Axial_DIN0207_L6.3mm_D2.5mm_P7.62mm_Horizontal, symbol Device:R
- J1: footprint atari:Atari2600_Cart_Slot_2x12_P2.54mm_Row5.50mm -> atari:Atari2600_Cart_Slot_2x12_P2.54mm_Row5.50mm_Guide
Connections:
- net +5V: now also F1.1; no longer C2.1, J1.23 (Pin_23)
- net GND: now also R6.2
- net CART_SENSE: now reaches A1.A0
- net CART_SENSE: now also R5.2
- net CART_PWR: now reaches A1.D10 (D10_CS)
- net CART_PWR: now also R3.1
- new net +5V_F: F1.2, Q1.3 (E), R4.1
- new net CART_5V: C2.1, J1.23 (Pin_23), Q1.1 (C), R5.1, R6.1
- new net Q_BASE: Q1.2 (B), R3.2, R4.2
- no-connect marks 30 -> 28

Commit message: Reset and read buttons on all boards (v1.2)
SW1 resets the Arduino, SW2 on A1 repeats the last dump; dump.py listen saves button dumps.

Co-Authored-By: Claude Opus 5.5 <noreply@anthropic.com>
Claude-Session: https://claude.ai/code/session_015VQCpzuZ22TPQEmx9cLrbH
Parts:
- added SW1: Reset, Button_Switch_THT:SW_PUSH_6mm, symbol Switch:SW_Push
- added SW2: Read, Button_Switch_THT:SW_PUSH_6mm, symbol Switch:SW_Push
Connections:
- net GND: now also SW1.2, SW2.2
- net READ: now reaches A1.A1
- net READ: now also SW2.1
- net RESET: now reaches A1.RST1 (RESET)
- net RESET: now also SW1.1
- no-connect marks 28 -> 26

Commit message: Uno/Nano: address bus via two 74HC595 on SPI, MCP23017 boards kept as variants
hal.h selects the MCP23017 with #define ADDR_MCP23017.

Co-Authored-By: Claude Opus 5.5 <noreply@anthropic.com>
Claude-Session: https://claude.ai/code/session_015VQCpzuZ22TPQEmx9cLrbH
Parts:
- removed R1, R2: 4k7, Resistor_THT:R_Axial_DIN0207_L6.3mm_D2.5mm_P7.62mm_Horizontal, symbol Device:R
- removed U1: MCP23017-E/SP, Package_DIP:DIP-28_W7.62mm_Socket, symbol Interface_Expansion:MCP23017_SP
- added C4: 100n, Capacitor_THT:C_Disc_D5.0mm_W2.5mm_P5.00mm, symbol Device:C
- added U1, U2: 74HC595, Package_DIP:DIP-16_W7.62mm_Socket, symbol 74xx:74HC595
Connections:
- net +5V: now also C4.1, U1.10 (~{SRCLR}), U1.16 (VCC), U2.10 (~{SRCLR}), U2.16 (VCC)
- net A0: now also U1.15 (QA)
- net A1: now also U1.1 (QB)
- net A10: now also U2.2 (QC)
- net A11: now also U2.3 (QD)
- net A12: now also U2.4 (QE)
- net A2: now also U1.2 (QC)
- net A3: now also U1.3 (QD)
- net A4: now also U1.4 (QE)
- net A5: now also U1.5 (QF)
- net A6: now also U1.6 (QG)
- net A7: now also U1.7 (QH)
- net A8: now also U2.15 (QA)
- net A9: now also U2.1 (QB)
- net GND: now also C4.2, U1.13 (~{OE}), U1.8 (GND), U2.13 (~{OE}), U2.8 (GND)
- net LATCH: now reaches A1.A2
- net LATCH: now also U1.12 (RCLK), U2.12 (RCLK)
- net MOSI: now reaches A1.D11
- net MOSI: now also U1.14 (SER)
- net SCK: now reaches A1.D13
- net SCK: now also U1.11 (SRCLK), U2.11 (SRCLK)
- net SCL: no longer names the net of A1.A5
- net SDA: no longer names the net of A1.A4
- new net SR_CHAIN: U1.9 (QH'), U2.14 (SER)
- no-connect marks 26 -> 22
Other:
- note added: "Aufsteckplatine fuer Arduino Uno R3. Adressbus A0-A12 ueber 2x 74HC595 (SPI: D11, D13, Latch A2), Datenbus D0-D7 an Uno D2-D9. Firmware: github.com/sfambach/arduino-atari2600-cart-reader - fambach.net"
- note removed: "Aufsteckplatine fuer Arduino Uno R3. Adressbus A0-A12 ueber MCP23017 (I2C 0x20), Datenbus D0-D7 an Uno D2-D9. Firmware: github.com/sfambach/arduino-atari2600-cart-reader - fambach.net"
